File: hardware/DigiCron.kicad_sch (KiCad schematic)
At the start: 6 parts, among them U100 MDBT50Q-U1MV2, U101 HCMS-3917, U102 HCMS-3917, X100 12401598E4#2A

Commit message: Add some sensor ICs to schematic
Parts:
- added U103: LTR-390UV-01, SMD6_LTR-390UV-01_LTO, symbol 2024-12-11_22-26-57:LTR-390UV-01
- added U104: ADXL345BCCZ-RL, LGA_CC-14-1_ADI, symbol ADXL345:ADXL345BCCZ-RL
- added U105: BMP280, Package_LGA:Bosch_LGA-8_2x2.5mm_P0.65mm_ClockwisePinNumbering, symbol Sensor_Pressure:BMP280
Connections:
- net +3V3: now also U103.1 (VDD), U104.1 (VDDI/O), U104.6 (VS), U104.7 (*CS), U105.6 (VDDIO), U105.8 (VDD)
- net GND: now also U103.3 (GND), U104.2 (GND), U104.4 (GND), U104.5 (GND), U105.1 (GND), U105.7 (GND)
- net SCL: now also U103.4 (SCL), U104.14 (SCL/SCLK), U105.4 (SCK)
- net SDA: now also U103.6 (SDA), U104.13 (SDA/SDI/SDIO), U105.3 (SDI)
- no-connect marks 19 -> 27

Commit message: Replace BMP280 with BME280 and add IR LED and JST connector
Parts:
- removed U105: BMP280, Package_LGA:Bosch_LGA-8_2x2.5mm_P0.65mm_ClockwisePinNumbering, symbol Sensor_Pressure:BMP280
- added D100: IR LED, LED_THT:LED_D5.0mm_Horizontal_O1.27mm_Z3.0mm_IRBlack, symbol Device:LED
- added J100: Conn_Receptacle_2P, Connector_JST:JST_PH_S2B-PH-SM4-TB_1x02-1MP_P2.00mm_Horizontal, symbol Connector:Conn_Receptacle_2P
- added U105: BME280, Package_LGA:Bosch_LGA-8_2.5x2.5mm_P0.65mm_ClockwisePinNumbering, symbol Sensor:BME280
- U101, U102: footprint DIP26_HCMS-290X-B_BRA -> HCMS-x91x:DIP26_HCMS-290X-B_BRA
- U103: footprint SMD6_LTR-390UV-01_LTO -> LTR390:SMD6_LTR-390UV-01_LTO
- U104: footprint LGA_CC-14-1_ADI -> ADXL345:LGA_CC-14-1_ADI
Connections:
- net +3V3: now also U105.6 (VDDIO), U105.8 (VDD)
- net GND: now also U105.1 (GND), U105.7 (GND)
- net SCL: now also U105.4 (SCK)
- net SDA: now also U105.3 (SDI)
- net JOY_UP: now reaches U100.5 (P1.12)
- net JOY_LEFT: now reaches U100.6 (P1.13)
- net JOY_RIGHT: now reaches U100.7 (P1.14)
- net JOY_DOWN: now reaches U100.8 (P1.15)
- net D10: no longer names the net of U100.16 (P0.27)
- net D11 renamed IR_OUT
- net D12 renamed IR_IN
- net D13 renamed JOY_SELECT
- net D5 renamed JOY_HOME
- net D6 renamed JOY_BACK
- net D9: no longer names the net of U100.19 (P0.26)
- no-connect marks 27 -> 23
