File: hardware/DigiCron.kicad_sch (KiCad schematic)
At the start: 20 parts, among them J100 Solder pad, J101 Solder pad, J102 Solder pad, J103 Solder pad, Q100 BSS138, Q101 AO3400A, U100 MDBT50Q-U1MV2, U101 HCMS-3917, U102 HCMS-3917, U104 ADXL345BCCZ-RL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

Commit message: Fix pin routing for battery power level sensing
Connections:
- net PIEZO_A: now also U100.13 (P0.28/AIN4); no longer U100.11 (P0.02/AIN0)
- net PIEZO_B: now also U100.11 (P0.02/AIN0); no longer U100.9 (P0.03/AIN1)
- net VDIV: now also U100.9 (P0.03/AIN1); no longer U100.16 (P0.27)
